File: eagle/pwm_techniques/logic/main.sch (EAGLE design)
At the start: 70 parts, among them IC1 7805T, U2 TLE2426ID, U3 LM358ADT, U4 TL494CD, U5 SN74HC04D, U6 TL494CD

Commit message: [ update ] logic schematics, connectors
Parts:
- added JP1: (no value), SparkFun:M02LOCK
- added JP2: (no value), SparkFun:M06LOCK
Connections:
- net GND: now also JP1.2, JP2.5
- net PWM_CTL_HI_0: now also JP2.3
- net PWM_CTL_HI_1: now also JP2.1
- net PWM_CTL_LO_0: now also JP2.4
- net PWM_CTL_LO_1: now also JP2.2
- net VBAT_12: now also JP1.1
- net VREG_10: now also JP2.6
Other:
- note added: "battery connector"
- note added: "output connector"
Changed lines of the file:
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@@
 <layer number="48" name="Document" color="7" fill="1" visible="yes" active="no"/>
 <layer number="49" name="Reference" color="7" fill="1" visible="yes" active="no"/>
+<layer number="50" name="dxf" color="7" fill="1" visible="no" active="no"/>
 <layer number="51" name="tDocu" color="7" fill="1" visible="yes" active="no"/>
 <layer number="52" name="bDocu" color="7" fill="1" visible="yes" active="no"/>
+<layer number="53" name="tGND_GNDA" color="7" fill="9" visible="no" active="no"/>
+<layer number="54" name="bGND_GNDA" color="1" fill="9" visible="no" active="no"/>
+<layer number="56" name="wert" color="7" fill="1" visible="no" active="no"/>
 <layer number="91" name="Nets" color="2" fill="1" visible="yes" active="yes"/>
 <layer number="92" name="Busses" color="1" fill="1" visible="yes" active="yes"/>
@@
 <layer number="97" name="Info" color="7" fill="1" visible="yes" active="yes"/>
 <layer number="98" name="Guide" color="6" fill="1" visible="yes" active="yes"/>
+<layer number="100" name="Muster" color="7" fill="1" visible="no" active="no"/>
+<layer number="101" name="Patch_Top" color="12" fill="4" visible="no" active="yes"/>
+<layer number="102" name="Vscore" color="7" fill="1" visible="no" active="yes"/>
+<layer number="103" name="tMap" color="7" fill="1" visible="no" active="yes"/>
+<layer number="104" name="Name" color="16" fill="1" visible="no" active="yes"/>
+<layer number="105" name="tPlate" color="7" fill="1" visible="no" active="yes"/>
+<layer number="106" name="bPlate" color="7" fill="1" visible="no" active="yes"/>
+<layer number="107" name="Crop" color="7" fill="1" visible="no" active="yes"/>
+<layer number="116" name="Patch_BOT" color="9" fill="4" visible="no" active="yes"/>
+<layer number="121" name="_tsilk" color="7" fill="1" visible="no" active="yes"/>
+<layer number="122" name="_bsilk" color="7" fill="1" visible="no" active="yes"/>
+<layer number="125" name="_tNames" color="7" fill="1" visible="no" active="yes"/>
+<layer number="144" name="Drill_legend" color="7" fill="1" visible="no" active="yes"/>
+<layer number="151" name="HeatSink" color="7" fill="1" visible="no" active="yes"/>
+<layer number="200" name="200bmp" color="1" fill="10" visible="no" active="yes"/>
+<layer number="201" name="201bmp" color="2" fill="10" visible="no" active="yes"/>
+<layer number="202" name="202bmp" color="3" fill="10" visible="no" active="yes"/>
+<layer number="203" name="203bmp" color="4" fill="10" visible="no" active="yes"/>
+<layer number="204" name="204bmp" color="5" fill="10" visible="no" active="yes"/>
+<layer number="205" name="205bmp" color="6" fill="10" visible="no" active="yes"/>
+<layer number="206" name="206bmp" color="7" fill="10" visible="no" active="yes"/>
+<layer number="207" name="207bmp" color="8" fill="10" visible="no" active="yes"/>
+<layer number="208" name="208bmp" color="9" fill="10" visible="no" active="yes"/>
+<layer number="209" name="209bmp" color="7" fill="1" visible="no" active="yes"/>
+<layer number="210" name="210bmp" color="7" fill="1" visible="no" active="yes"/>
+<layer number="211" name="211bmp" color="7" fill="1" visible="no" active="yes"/>
+<layer number="212" name="212bmp" color="7" fill="1" visible="no" active="yes"/>
+<layer number="213" name="213bmp" color="7" fill="1" visible="no" active="yes"/>
+<layer number="214" name="214bmp" color="7" fill="1" visible="no" active="yes"/>
+<layer number="215" name="215bmp" color="7" fill="1" visible="no" active="yes"/>
+<layer number="216" name="216bmp" color="7" fill="1" visible="no" active="yes"/>
+<layer number="217" name="217bmp" color="18" fill="1" visible="no" active="no"/>
+<layer number="218" name="218bmp" color="19" fill="1" visible="no" active="no"/>
+<layer number="219" name="219bmp" color="20" fill="1" visible="no" active="no"/>
+<layer number="220" name="220bmp" color="21" fill="1" visible="no" active="no"/>
+<layer number="221" name="221bmp" color="22" fill="1" visible="no" active="no"/>
+<layer number="222" name="222bmp" color="23" fill="1" visible="no" active="no"/>
+<layer number="223" name="223bmp" color="24" fill="1" visible="no" active="no"/>
+<layer number="224" name="224bmp" color="25" fill="1" visible="no" active="no"/>
+<layer number="250" name="Descript" color="3" fill="1" visible="no" active="no"/>
+<layer number="251" name="SMDround" color="12" fill="11" visible="no" active="no"/>
+<layer number="254" name="cooling" color="7" fill="1" visible="no" active="yes"/>
 </layers>
 <schematic xreflabel="%F%N/%S.%C%R" xrefpart="/%S.%C%R">
@@
 <part name="IC1" library="linear" deviceset="78*" device="T" technology="05"/>
 <part name="LM2940T_10" library="linear" deviceset="78*" device="T" technology="05"/>
+<part name="JP1" library="SparkFun" deviceset="M02" device="LOCK"/>
+<part name="JP2" library="SparkFun" deviceset="M06" device="LOCK"/>
 </parts>
 <sheets>
@@
 <text x="454.66" y="101.6" size="1.778" layer="97">pwm controller stage</text>
 <text x="-20.32" y="86.36" size="1.778" layer="97">WARNING: actually a LM2940T, 7805T used only for footprint</text>
+<text x="-60.96" y="101.6" size="1.778" layer="97">battery connector</text>
+<text x="551.18" y="101.6" size="1.778" layer="97">output connector</text>
 </plain>
 <instances>
@@
 <instance part="IC1" gate="A1" x="12.7" y="33.02"/>
 <instance part="LM2940T_10" gate="A1" x="12.7" y="76.2"/>
+<instance part="JP1" gate="G$1" x="-43.18" y="78.74" rot="R180"/>
+<instance part="JP2" gate="G$1" x="548.64" y="68.58"/>
 </instances>
 <busses>
@@
 <junction x="-10.16" y="76.2"/>
 <pinref part="LM2940T_10" gate="A1" pin="VI"/>
+</segment>
+<segment>
+<pinref part="JP1" gate="G$1" pin="1"/>
+<wire x1="-50.8" y1="78.74" x2="-63.5" y2="78.74" width="0.1524" layer="91"/>
+<label x="-63.5" y="78.74" size="1.778" layer="95"/>
 </segment>
 </net>
@@
 <junction x="43.18" y="76.2"/>
 <pinref part="LM2940T_10" gate="A1" pin="VO"/>
+</segment>
+<segment>
+<wire x1="553.72" y1="76.2" x2="574.04" y2="76.2" width="0.1524" layer="91"/>
+<pinref part="JP2" gate="G$1" pin="6"/>
+<label x="556.26" y="76.2" size="1.778" layer="95"/>
 </segment>
 </net>
@@
 <pinref part="LM2940T_10" gate="A1" pin="GND"/>
 </segment>
+<segment>
+<pinref part="JP1" gate="G$1" pin="2"/>
+<wire x1="-50.8" y1="76.2" x2="-63.5" y2="76.2" width="0.1524" layer="91"/>
+<label x="-63.5" y="76.2" size="1.778" layer="95"/>
+</segment>
+<segment>
+<pinref part="JP2" gate="G$1" pin="5"/>
+<wire x1="553.72" y1="73.66" x2="574.04" y2="73.66" width="0.1524" layer="91"/>
+<label x="556.26" y="73.66" size="1.778" layer="95"/>
+</segment>
 </net>
 <net name="VSPLIT_GND" class="0">
@@
 <label x="429.26" y="-96.52" size="1.778" layer="95"/>
 </segment>
+<segment>
+<pinref part="JP2" gate="G$1" pin="4"/>
+<wire x1="574.04" y1="71.12" x2="553.72" y2="71.12" width="0.1524" layer="91"/>
+<label x="556.26" y="71.12" size="1.778" layer="95"/>
+</segment>
 </net>
 <net name="N$4" class="0">
@@
 <junction x="490.22" y="2.54"/>
 </segment>
+<segment>
+<pinref part="JP2" gate="G$1" pin="2"/>
+<wire x1="574.04" y1="66.04" x2="553.72" y2="66.04" width="0.1524" layer="91"/>
+<label x="556.26" y="66.04" size="1.778" layer="95"/>
+</segment>
 </net>
 <net name="PWM_CTL_HI_0" class="0">
@@
 <label x="487.68" y="-91.44" size="1.778" layer="95"/>
 </segment>
+<segment>
+<pinref part="JP2" gate="G$1" pin="3"/>
+<wire x1="574.04" y1="68.58" x2="553.72" y2="68.58" width="0.1524" layer="91"/>
+<label x="556.26" y="68.58" size="1.778" layer="95"/>
+</segment>
 </net>
 <net name="PWM_CTL_HI_1" class="0">
@@
 <label x="487.68" y="-93.98" size="1.778" layer="95"/>
 </segment>
-</net>
+<segment>
+<pinref part="JP2" gate="G$1" pin="1"/>
+<wire x1="574.04" y1="63.5" x2="553.72" y2="63.5" width="0.1524" layer="91"/>
+<label x="556.26" y="63.5" size="1.778" layer="95"/>
+</segment>
+</net>
